File: pcb/Particlematrix10x5.brd (EAGLE design)
At the start: 101.6 x 53.3 mm, 68 parts, among them IC1 4017D

Commit message: Cleanup in schematic
Routing:
- net N$9: track 221.2 -> 219.4 mm
Changed lines of the file:
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@@
 </signal>
 <signal name="N$6">
-<contactref element="IC1" pad="16"/>
 <contactref element="PCB1" pad="5V"/>
-<wire x1="-12.1666" y1="64.135" x2="-12.1666" y2="74.1934" width="0.2032" layer="1"/>
 <wire x1="-12.1666" y1="74.1934" x2="-8.89" y2="77.47" width="0.2032" layer="1"/>
 <wire x1="-8.89" y1="77.47" x2="92.71" y2="77.47" width="0.2032" layer="1"/>
@@
 <wire x1="59.69" y1="31.75" x2="59.69" y2="27.94" width="0.2032" layer="16"/>
 <via x="93.98" y="35.56" extent="1-16" drill="0.6" shape="square"/>
+<contactref element="IC1" pad="16"/>
+<wire x1="-12.1666" y1="74.1934" x2="-12.1666" y2="64.135" width="0.2032" layer="1"/>
 </signal>
 <signal name="N$9">
-<contactref element="IC1" pad="8"/>
 <contactref element="PCB1" pad="GND.."/>
-<wire x1="-18.3134" y1="55.245" x2="-16.51" y2="55.245" width="0.2032" layer="1"/>
 <wire x1="-16.51" y1="55.245" x2="-15.875" y2="55.88" width="0.2032" layer="1"/>
 <wire x1="-15.875" y1="55.88" x2="-15.875" y2="66.04" width="0.2032" layer="16"/>
@@
 <via x="-15.875" y="55.88" extent="1-16" drill="0.6" shape="square"/>
 <via x="-15.875" y="66.04" extent="1-16" drill="0.6" shape="square"/>
+<contactref element="IC1" pad="8"/>
+<wire x1="-18.3134" y1="55.245" x2="-16.51" y2="55.245" width="0" layer="19" extent="1-1"/>
 </signal>
 <signal name="RAW">
